File: pwm_circuit.kicad_sch (KiCad schematic)
At the start: 6 parts

Commit message: added foot prints
Parts:
- removed C?: C_Polarized_US, symbol Device:C_Polarized_US
- added C1: 1uF, Capacitor_Tantalum_SMD:CP_EIA-6032-15_Kemet-U, symbol Device:C_Polarized_Small_US
- R11, R12, R13, R14: renamed from R?; footprint (none) -> Resistor_SMD:R_0603_1608Metric
- gave numbers to parts that had none: 1
Connections:
- net GND: now also C1.2
- net PWM_vcc: now also C1.1
Changed lines of the file:
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@@
     (stroke (width 0) (type default) (color 0 0 0 0))
   )
-  (wire (pts (xy 203.835 99.06) (xy 203.835 115.57))
+  (wire (pts (xy 203.835 96.52) (xy 203.835 115.57))
     (stroke (width 0) (type default) (color 0 0 0 0))
   )
@@
   (symbol (lib_id "Device:R") (at 179.07 93.98 90) (unit 1)
     (in_bom yes) (on_board yes) (fields_autoplaced)
-    (property "Reference" "R?" (id 0) (at 179.07 88.265 90))
+    (property "Reference" "R14" (id 0) (at 179.07 88.265 90))
     (property "Value" "R" (id 1) (at 179.07 90.805 90))
-    (property "Footprint" "" (id 2) (at 179.07 95.758 90)
+    (property "Footprint" "Resistor_SMD:R_0603_1608Metric" (id 2) (at 179.07 95.758 90)
       (effects (font (size 1.27 1.27)) hide)
     )
@@
   (symbol (lib_id "power:+5V") (at 168.91 85.09 90) (unit 1)
     (in_bom yes) (on_board yes) (fields_autoplaced)
-    (property "Reference" "#PWR?" (id 0) (at 172.72 85.09 0)
+    (property "Reference" "#PWR07" (id 0) (at 172.72 85.09 0)
       (effects (font (size 1.27 1.27)) hide)
     )
@@
     (pin "1")
   )
-  (symbol (lib_id "Device:C_Polarized_US") (at 203.835 95.25 0) (unit 1)
-    (in_bom yes) (on_board yes) (fields_autoplaced)
-    (property "Reference" "C?" (id 0) (at 207.645 93.3449 0)
-      (effects (font (size 1.27 1.27)) (justify left))
-    )
-    (property "Value" "C_Polarized_US" (id 1) (at 207.645 95.8849 0)
-      (effects (font (size 1.27 1.27)) (justify left))
-    )
-    (property "Footprint" "" (id 2) (at 203.835 95.25 0)
-      (effects (font (size 1.27 1.27)) hide)
-    )
-    (property "Datasheet" "~" (id 3) (at 203.835 95.25 0)
-      (effects (font (size 1.27 1.27)) hide)
-    )
-    (pin "1")
-    (pin "2")
-  )
   (symbol (lib_id "Device:R") (at 171.45 64.77 0) (unit 1)
     (in_bom yes) (on_board yes) (fields_autoplaced)
-    (property "Reference" "R?" (id 0) (at 173.99 63.4999 0)
+    (property "Reference" "R12" (id 0) (at 173.99 63.4999 0)
       (effects (font (size 1.27 1.27)) (justify left))
     )
@@
       (effects (font (size 1.27 1.27)) (justify left))
     )
-    (property "Footprint" "" (id 2) (at 169.672 64.77 90)
+    (property "Footprint" "Resistor_SMD:R_0603_1608Metric" (id 2) (at 169.672 64.77 90)
       (effects (font (size 1.27 1.27)) hide)
     )
@@
   (symbol (lib_id "Transistor_FET:2N7002") (at 154.94 73.025 270) (unit 1)
     (in_bom yes) (on_board yes) (fields_autoplaced)
-    (property "Reference" "Q?" (id 0) (at 154.94 80.645 90))
+    (property "Reference" "Q1" (id 0) (at 154.94 80.645 90))
     (property "Value" "2N7002" (id 1) (at 154.94 83.185 90))
     (property "Footprint" "Package_TO_SOT_SMD:SOT-23" (id 2) (at 153.035 78.105 0)
@@
   (symbol (lib_id "Device:R") (at 179.07 85.09 90) (unit 1)
     (in_bom yes) (on_board yes) (fields_autoplaced)
-    (property "Reference" "R?" (id 0) (at 179.07 79.375 90))
+    (property "Reference" "R13" (id 0) (at 179.07 79.375 90))
     (property "Value" "R" (id 1) (at 179.07 81.915 90))
-    (property "Footprint" "" (id 2) (at 179.07 86.868 90)
+    (property "Footprint" "Resistor_SMD:R_0603_1608Metric" (id 2) (at 179.07 86.868 90)
       (effects (font (size 1.27 1.27)) hide)
     )
@@
     (pin "2")
   )
+  (symbol (lib_id "Device:C_Polarized_Small_US") (at 203.835 93.98 0) (unit 1)
+    (in_bom yes) (on_board yes) (fields_autoplaced)
+    (property "Reference" "C1" (id 0) (at 206.375 92.2781 0)
+      (effects (font (size 1.27 1.27)) (justify left))
+    )
+    (property "Value" "1uF" (id 1) (at 206.375 94.8181 0)
+      (effects (font (size 1.27 1.27)) (justify left))
+    )
+    (property "Footprint" "Capacitor_Tantalum_SMD:CP_EIA-6032-15_Kemet-U" (id 2) (at 203.835 93.98 0)
+      (effects (font (size 1.27 1.27)) hide)
+    )
+    (property "Datasheet" "~" (id 3) (at 203.835 93.98 0)
+      (effects (font (size 1.27 1.27)) hide)
+    )
+    (pin "1")
+    (pin "2")
+  )
   (symbol (lib_id "power:+3V3") (at 168.91 93.98 90) (unit 1)
     (in_bom yes) (on_board yes) (fields_autoplaced)
-    (property "Reference" "#PWR?" (id 0) (at 172.72 93.98 0)
+    (property "Reference" "#PWR08" (id 0) (at 172.72 93.98 0)
       (effects (font (size 1.27 1.27)) hide)
     )
@@
   (symbol (lib_id "Device:R") (at 139.065 65.405 0) (unit 1)
     (in_bom yes) (on_board yes) (fields_autoplaced)
-    (property "Reference" "R?" (id 0) (at 140.97 64.1349 0)
+    (property "Reference" "R11" (id 0) (at 140.97 64.1349 0)
       (effects (font (size 1.27 1.27)) (justify left))
     )
@@
       (effects (font (size 1.27 1.27)) (justify left))
     )
-    (property "Footprint" "" (id 2) (at 137.287 65.405 90)
+    (property "Footprint" "Resistor_SMD:R_0603_1608Metric" (id 2) (at 137.287 65.405 90)
       (effects (font (size 1.27 1.27)) hide)
     )
@@
   (symbol (lib_id "power:+3V3") (at 139.065 55.245 0) (unit 1)
     (in_bom yes) (on_board yes) (fields_autoplaced)
-    (property "Reference" "#PWR?" (id 0) (at 139.065 59.055 0)
+    (property "Reference" "#PWR06" (id 0) (at 139.065 59.055 0)
       (effects (font (size 1.27 1.27)) hide)
     )
@@
   (symbol (lib_id "power:+5V") (at 171.45 55.245 0) (unit 1)
     (in_bom yes) (on_board yes) (fields_autoplaced)
-    (property "Reference" "#PWR?" (id 0) (at 171.45 59.055 0)
+    (property "Reference" "#PWR09" (id 0) (at 171.45 59.055 0)
       (effects (font (size 1.27 1.27)) hide)
     )
@@
   (symbol (lib_id "power:GND") (at 174.625 115.57 0) (unit 1)
     (in_bom yes) (on_board yes) (fields_autoplaced)
-    (property "Reference" "#PWR?" (id 0) (at 174.625 121.92 0)
-      (effects (font (size 1.27 1.27)) hide)
-    )
+    (property "Reference" "#PWR010" (id 0) (at 174.625 121.92 0)
+      (effects (font (size 1.27 1.27)) hide)
+    )
