File: qei_circuit.kicad_sch (KiCad schematic)
At the start: 7 parts

Commit message: added foot prints
Parts:
- removed C?: 1u, symbol Device:C_Polarized_US
- added C3: 1uF, symbol Device:C_Polarized_Small_US
- R19, R20, R21, R22: renamed from R?; footprint (none) -> Resistor_SMD:R_0603_1608Metric
- gave numbers to parts that had none: 2
Connections:
- net +5V: now also C3.1
- net GND: now also C3.2
Changed lines of the file:
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@@
     (stroke (width 0) (type default) (color 0 0 0 0))
   )
-  (wire (pts (xy 171.45 109.855) (xy 171.45 117.475))
+  (wire (pts (xy 171.45 107.315) (xy 171.45 117.475))
     (stroke (width 0) (type default) (color 0 0 0 0))
   )
@@
   (symbol (lib_id "power:GND") (at 96.52 111.125 0) (unit 1)
     (in_bom yes) (on_board yes) (fields_autoplaced)
-    (property "Reference" "#PWR?" (id 0) (at 96.52 117.475 0)
+    (property "Reference" "#PWR019" (id 0) (at 96.52 117.475 0)
       (effects (font (size 1.27 1.27)) hide)
     )
@@
   (symbol (lib_id "power:+5V") (at 73.025 142.875 180) (unit 1)
     (in_bom yes) (on_board yes) (fields_autoplaced)
-    (property "Reference" "#PWR?" (id 0) (at 73.025 139.065 0)
+    (property "Reference" "#PWR017" (id 0) (at 73.025 139.065 0)
       (effects (font (size 1.27 1.27)) hide)
     )
@@
   (symbol (lib_id "Transistor_FET:2N7002") (at 102.235 125.095 0) (unit 1)
     (in_bom yes) (on_board yes) (fields_autoplaced)
-    (property "Reference" "Q?" (id 0) (at 107.95 123.8249 0)
+    (property "Reference" "Q4" (id 0) (at 107.95 123.8249 0)
       (effects (font (size 1.27 1.27)) (justify left))
     )
@@
   (symbol (lib_id "Transistor_FET:2N7002") (at 93.98 99.695 0) (unit 1)
     (in_bom yes) (on_board yes) (fields_autoplaced)
-    (property "Reference" "Q?" (id 0) (at 99.695 98.4249 0)
+    (property "Reference" "Q3" (id 0) (at 99.695 98.4249 0)
       (effects (font (size 1.27 1.27)) (justify left))
     )
@@
   (symbol (lib_id "Device:R") (at 72.39 92.71 0) (unit 1)
     (in_bom yes) (on_board yes) (fields_autoplaced)
-    (property "Reference" "R?" (id 0) (at 74.93 91.4399 0)
+    (property "Reference" "R19" (id 0) (at 74.93 91.4399 0)
       (effects (font (size 1.27 1.27)) (justify left))
     )
@@
       (effects (font (size 1.27 1.27)) (justify left))
     )
-    (property "Footprint" "" (id 2) (at 70.612 92.71 90)
+    (property "Footprint" "Resistor_SMD:R_0603_1608Metric" (id 2) (at 70.612 92.71 90)
       (effects (font (size 1.27 1.27)) hide)
     )
@@
   (symbol (lib_id "Device:R") (at 104.775 114.3 0) (unit 1)
     (in_bom yes) (on_board yes) (fields_autoplaced)
-    (property "Reference" "R?" (id 0) (at 106.68 113.0299 0)
+    (property "Reference" "R22" (id 0) (at 106.68 113.0299 0)
       (effects (font (size 1.27 1.27)) (justify left))
     )
@@
       (effects (font (size 1.27 1.27)) (justify left))
     )
-    (property "Footprint" "" (id 2) (at 102.997 114.3 90)
+    (property "Footprint" "Resistor_SMD:R_0603_1608Metric" (id 2) (at 102.997 114.3 90)
       (effects (font (size 1.27 1.27)) hide)
     )
@@
   (symbol (lib_id "power:+5V") (at 180.975 95.885 0) (unit 1)
     (in_bom yes) (on_board yes) (fields_autoplaced)
-    (property "Reference" "#PWR?" (id 0) (at 180.975 99.695 0)
+    (property "Reference" "#PWR022" (id 0) (at 180.975 99.695 0)
       (effects (font (size 1.27 1.27)) hide)
     )
@@
   (symbol (lib_id "Device:R") (at 73.025 131.445 0) (unit 1)
     (in_bom yes) (on_board yes) (fields_autoplaced)
-    (property "Reference" "R?" (id 0) (at 74.93 130.1749 0)
+    (property "Reference" "R20" (id 0) (at 74.93 130.1749 0)
       (effects (font (size 1.27 1.27)) (justify left))
     )
@@
       (effects (font (size 1.27 1.27)) (justify left))
     )
-    (property "Footprint" "" (id 2) (at 71.247 131.445 90)
+    (property "Footprint" "Resistor_SMD:R_0603_1608Metric" (id 2) (at 71.247 131.445 90)
       (effects (font (size 1.27 1.27)) hide)
     )
@@
   (symbol (lib_id "Device:R") (at 96.52 85.725 0) (unit 1)
     (in_bom yes) (on_board yes) (fields_autoplaced)
-    (property "Reference" "R?" (id 0) (at 99.06 84.4549 0)
+    (property "Reference" "R21" (id 0) (at 99.06 84.4549 0)
       (effects (font (size 1.27 1.27)) (justify left))
     )
@@
       (effects (font (size 1.27 1.27)) (justify left))
     )
-    (property "Footprint" "" (id 2) (at 94.742 85.725 90)
+    (property "Footprint" "Resistor_SMD:R_0603_1608Metric" (id 2) (at 94.742 85.725 90)
       (effects (font (size 1.27 1.27)) hide)
     )
@@
     (pin "2")
   )
-  (symbol (lib_id "Device:C_Polarized_US") (at 171.45 106.045 0) (unit 1)
-    (in_bom yes) (on_board yes) (fields_autoplaced)
-    (property "Reference" "C?" (id 0) (at 175.26 104.1399 0)
-      (effects (font (size 1.27 1.27)) (justify left))
-    )
-    (property "Value" "1u" (id 1) (at 175.26 106.6799 0)
-      (effects (font (size 1.27 1.27)) (justify left))
-    )
-    (property "Footprint" "" (id 2) (at 171.45 106.045 0)
-      (effects (font (size 1.27 1.27)) hide)
-    )
-    (property "Datasheet" "~" (id 3) (at 171.45 106.045 0)
-      (effects (font (size 1.27 1.27)) hide)
-    )
-    (pin "1")
-    (pin "2")
-  )
   (symbol (lib_id "power:GND") (at 180.975 121.92 0) (unit 1)
     (in_bom yes) (on_board yes) (fields_autoplaced)
-    (property "Reference" "#PWR?" (id 0) (at 180.975 128.27 0)
+    (property "Reference" "#PWR023" (id 0) (at 180.975 128.27 0)
       (effects (font (size 1.27 1.27)) hide)
     )
@@
   (symbol (lib_id "power:GND") (at 104.775 142.875 0) (unit 1)
     (in_bom yes) (on_board yes) (fields_autoplaced)
-    (property "Reference" "#PWR?" (id 0) (at 104.775 149.225 0)
+    (property "Reference" "#PWR021" (id 0) (at 104.775 149.225 0)
       (effects (font (size 1.27 1.27)) hide)
     )
@@
   (symbol (lib_id "power:+3V3") (at 96.52 76.835 0) (unit 1)
     (in_bom yes) (on_board yes) (fields_autoplaced)
-    (property "Reference" "#PWR?" (id 0) (at 96.52 80.645 0)
+    (property "Reference" "#PWR018" (id 0) (at 96.52 80.645 0)
       (effects (font (size 1.27 1.27)) hide)
     )
@@
   (symbol (lib_id "power:+5V") (at 72.39 83.185 0) (unit 1)
     (in_bom yes) (on_board yes) (fields_autoplaced)
-    (property "Reference" "#PWR?" (id 0) (at 72.39 86.995 0)
+    (property "Reference" "#PWR016" (id 0) (at 72.39 86.995 0)
       (effects (font (size 1.27 1.27)) hide)
     )
@@
     (pin "1")
   )
+  (symbol (lib_id "Device:C_Polarized_Small_US") (at 171.45 104.775 0) (unit 1)
+    (in_bom yes) (on_board yes) (fields_autoplaced)
+    (property "Reference" "C3" (id 0) (at 173.99 103.0731 0)
+      (effects (font (size 1.27 1.27)) (justify left))
+    )
+    (property "Value" "1uF" (id 1) (at 173.99 105.6131 0)
+      (effects (font (size 1.27 1.27)) (justify left))
+    )
+    (property "Footprint" "" (id 2) (at 171.45 104.775 0)
+      (effects (font (size 1.27 1.27)) hide)
+    )
+    (property "Datasheet" "~" (id 3) (at 171.45 104.775 0)
+      (effects (font (size 1.27 1.27)) hide)
+    )
+    (pin "1")
+    (pin "2")
+  )
   (symbol (lib_id "power:+3V3") (at 104.775 109.22 0) (unit 1)
     (in_bom yes) (on_board yes) (fields_autoplaced)
-    (property "Reference" "#PWR?" (id 0) (at 104.775 113.03 0)
-      (effects (font (size 1.27 1.27)) hide)
-    )
+    (property "Reference" "#PWR020" (id 0) (at 104.775 113.03 0)
+      (effects (font (size 1.27 1.27)) hide)
+    )

Commit message: added 3.3v regulator
Parts:
- C3: footprint (none) -> Capacitor_Tantalum_SMD:CP_EIA-6032-15_Kemet-U
Changed lines of the file:
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@@
       (effects (font (size 1.27 1.27)) (justify left))
     )
-    (property "Footprint" "" (id 2) (at 171.45 104.775 0)
+    (property "Footprint" "Capacitor_Tantalum_SMD:CP_EIA-6032-15_Kemet-U" (id 2) (at 171.45 104.775 0)
       (effects (font (size 1.27 1.27)) hide)
     )
